File: Sweep v2.2 NoLogo/sweepv2-nologo_plate.kicad_pcb (KiCad board)
At the start: 2 copper layers, 105 x 86.9 mm, 17 parts, among them SW10 SW_Push, SW11 SW_Push, SW12 SW_Push, SW14 SW_Push, SW15 SW_Push, SW16 SW_Push, SW17 SW_Push, SW18 SW_Push, SW2 SW_Push, SW20 SW_Push, SW21 SW_Push, SW3 SW_Push, SW4 SW_Push, SW5 SW_Push, SW6 SW_Push, SW8 SW_Push, SW9 SW_Push

Commit message: revert: feat(sweep_v2_2_nologo): fill plate zones
This reverts commit b860a7d7b3753e3c2efd8507f68df48834ce2f9f.
Parts:
- moved SW15 37.3 mm to (40.0, 63.0)
- moved SW9 37.3 mm to (40.0, 46.0)
- moved SW14 37.3 mm to (22.0, 75.0)
- moved SW2 37.3 mm to (22.0, 41.0)
- moved SW21 37.3 mm to (86.0, 81.7)
- moved SW3 37.3 mm to (40.0, 29.0)
- moved SW8 37.3 mm to (22.0, 58.0)
- moved SW10 37.3 mm to (58.0, 39.1)
- moved SW11 37.3 mm to (76.0, 44.5)
- moved SW12 37.3 mm to (94.0, 47.0)
- moved SW16 37.3 mm to (58.0, 56.1)
- moved SW17 37.3 mm to (76.0, 61.5)
- moved SW18 37.3 mm to (94.0, 64.0)
- moved SW20 37.3 mm to (104.5, 89.7)
- moved SW4 37.3 mm to (58.0, 22.0)
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Routing:
- removed copper zone on B.Cu, net gnd
- removed copper zone on F.Cu, net gnd
Other:
- net class Default added: clearance 0.2, trace_width 0.25, via_dia 0.8, via_drill 0.4

Commit message: feat(sweep_v2_2_nologo): fill plate zones
Due to my KiCad inexperience, this commit was done by:

1. Open `Sweep v2.2 NoLogo/sweepv2-nologo_plate.kicad_pcb` and `Sweep
   v2.2 High/sweep-high_plate.kicad_pcb` in seperate KiCad instances.
2. Delete plate in `Sweep v2.2 High/sweep-high_plate.kicad_pcb`.
3. Copy plate in `Sweep v2.2 NoLogo/sweepv2-nologo_plate.kicad_pcb` to
   `Sweep v2.2 High/sweep-high_plate.kicad_pcb`.
4. Fill all zones in `Sweep v2.2 High/sweep-high_plate.kicad_pcb`.
5. Save changes in `Sweep v2.2 High/sweep-high_plate.kicad_pcb` and
   discard changes in `Sweep v2.2
   NoLogo/sweepv2-nologo_plate.kicad_pcb`.
6. Close both KiCad instances.
7. Run `mv 'Sweep v2.2 High/sweep-high_plate.kicad_pcb' 'Sweep v2.2
   NoLogo/sweepv2-nologo_plate.kicad_pcb'`.
8. Run `git restore 'Sweep v2.2 High/sweep-high_plate.kicad_pcb'`.
Parts:
- moved SW15 37.3 mm to (58.4, 95.4)
- moved SW9 37.3 mm to (58.4, 78.4)
- moved SW14 37.3 mm to (40.4, 107.4)
- moved SW2 37.3 mm to (40.4, 73.4)
- moved SW21 37.3 mm to (104.3, 114.1)
- moved SW3 37.3 mm to (58.4, 61.4)
- moved SW8 37.3 mm to (40.4, 90.4)
- moved SW10 37.3 mm to (76.4, 71.6)
- moved SW11 37.3 mm to (94.4, 76.9)
- moved SW12 37.3 mm to (112.4, 79.4)
- moved SW16 37.3 mm to (76.4, 88.6)
- moved SW17 37.3 mm to (94.4, 93.9)
- moved SW18 37.3 mm to (112.4, 96.5)
- moved SW20 37.3 mm to (122.9, 122.1)
- moved SW4 37.3 mm to (76.4, 54.4)
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Routing:
- added copper zone on B.Cu, net gnd
- added copper zone on F.Cu, net gnd
Other:
- net class Default removed
